File: Eagle/V2.2/PowerMeter.sch (EAGLE design)
At the start: 56 parts, among them IC1 74HC138D, IC2 4052D, IC3 CS5463, Q1 4.096MHz, T1 TV16E, T2 TV16E, T3 TV16E, X1 RASPI_BOARD_B+_E4

Commit message: Cleaned up some thing
cleaned up traces, made 3.5mm connectors, caps & diode SMD, put everything on same side of boards (may need to put resistor arrays back on the underside of the main board).
Parts:
- C5: value 220uF -> 220uF / 865080345012; device adafruit:CPOL-USE2,5-6E -> rcl:CPOL-USUD-6,3X7,7
- D1: value P6KE6.8A -> SMBJP6KE6.8A-TP; device diode:P6KEXXA -> SamacSys_Parts:B340A-13-F; PARTNO P6KE6.8A -> (none)
- Q1: device crystal:CRYSTALHC49S -> SamacSys_Parts:9C-8.000MAAJ-T
Connections:
- net 5V: now also D1.K; no longer D1.C
