File: Eagle/V2.2/PowerMeterCurrent.sch (EAGLE design)
At the start: 59 parts, among them IC1 4067D, IC2 4514D, X1 STEREOJACK, X10 STEREOJACK, X11 STEREOJACK, X12 STEREOJACK, X13 STEREOJACK, X14 STEREOJACK, X15 STEREOJACK, X16 STEREOJACK, X2 STEREOJACK, X3 STEREOJACK, X4 STEREOJACK, X5 STEREOJACK, X6 STEREOJACK, X7 STEREOJACK, X8 STEREOJACK, X9 STEREOJACK

Commit message: Cleaned up some thing
cleaned up traces, made 3.5mm connectors, caps & diode SMD, put everything on same side of boards (may need to put resistor arrays back on the underside of the main board).
Parts:
- removed X1, X10, X11, X12, X13, X14, X15, X16, X2, X3, X4, X5, X6, X7, X8, X9: STEREOJACK, adafruit:STEREOJACK
- added J1, J10, J11, J12, J13, J14, J15, J16, J2, J3, J4, J5, J6, J7, J8, J9: SJ2-35813B-SMT-TR, SJ2-35813B-SMT-TR:SJ2-35813B-SMT-TR
Connections:
- removed net N$12: R1.2, R10.2, R11.2, R12.2, R13.2, R14.2, R15.2, R16.2, R2.2, R3.2, R4.2, R5.2, R6.2, R7.2, R8.2, R9.2, SV1.16, X1.1, X1.4, X10.1, X10.4, X11.1, X11.4, X12.1, X12.4, X13.1, X13.4, X14.1, X14.4, X15.1, X15.4, X16.1, X16.4, X2.1, X2.4, X3.1, X3.4, X4.1, X4.4, X5.1, X5.4, X6.1, X6.4, X7.1, X7.4, X8.1, X8.4, X9.1, X9.4
- new net CT-: J1.SLEEVE, J1.TIP_SWITCH, J10.SLEEVE, J10.TIP_SWITCH, J11.SLEEVE, J11.TIP_SWITCH, J12.SLEEVE, J12.TIP_SWITCH, J13.SLEEVE, J13.TIP_SWITCH, J14.SLEEVE, J14.TIP_SWITCH, J15.SLEEVE, J15.TIP_SWITCH, J16.SLEEVE, J16.TIP_SWITCH, J2.SLEEVE, J2.TIP_SWITCH, J3.SLEEVE, J3.TIP_SWITCH, J4.SLEEVE, J4.TIP_SWITCH, J5.SLEEVE, J5.TIP_SWITCH, J6.SLEEVE, J6.TIP_SWITCH, J7.SLEEVE, J7.TIP_SWITCH, J8.SLEEVE, J8.TIP_SWITCH, J9.SLEEVE, J9.TIP_SWITCH, R1.2, R10.2, R11.2, R12.2, R13.2, R14.2, R15.2, R16.2, R2.2, R3.2, R4.2, R5.2, R6.2, R7.2, R8.2, R9.2, SV1.16
- net N$18: now also J5.TIP; no longer X5.5
- net N$20: now also J1.TIP; no longer X1.5
- net N$22: now also J2.TIP; no longer X2.5
- net N$23: now also J3.TIP; no longer X3.5
- net N$24: now also J4.TIP; no longer X4.5
- net N$25: now also J6.TIP; no longer X6.5
- net N$26: now also J7.TIP; no longer X7.5
- net N$28: now also J8.TIP; no longer X8.5
- net N$29: now also J9.TIP; no longer X9.5
- net N$50: now also J10.TIP; no longer X10.5
- net N$51: now also J11.TIP; no longer X11.5
- net N$58: now also J12.TIP; no longer X12.5
- net N$59: now also J14.TIP; no longer X14.5
- net N$60: now also J15.TIP; no longer X15.5
- net N$66: now also J13.TIP; no longer X13.5
- net N$68: now also J16.TIP; no longer X16.5
